Commit message: Complete robot audio, motion, and hardware updates

File: Emulator/sesame-robot-sim/app/robot.urdf (robot description, URDF)
Before this commit: robot onshape, 25 links, 24 joints
Joints:
- joint l3_p1_frame: origin xyz=0.001905 0.04706 -0.0199857 rpy=-1.5708 1.5708 0 -> xyz=0.001905 0.0638208 -0.0199857 rpy=-1.5708 1.5708 0
- joint l3_p2_frame: origin xyz=0.001905 0.04706 -0.0120344 rpy=-1.5708 1.5708 0 -> xyz=0.001905 0.0638208 -0.0120344 rpy=-1.5708 1.5708 0
- joint l3_p3_frame: origin xyz=-0.00508 0.04706 -0.0199857 rpy=-1.5708 1.5708 0 -> xyz=-0.00508 0.0638208 -0.0199857 rpy=-1.5708 1.5708 0
- joint l3_p4_frame: origin xyz=-0.00508 0.04706 -0.0123397 rpy=-1.5708 1.5708 0 -> xyz=-0.00508 0.0638208 -0.0123397 rpy=-1.5708 1.5708 0
- joint r3_p1_frame: origin xyz=0.001905 -0.04706 -0.0195906 rpy=1.5708 1.5708 0 -> xyz=0.001905 -0.0638208 -0.0195906 rpy=1.5708 1.5708 0
- joint r3_p2_frame: origin xyz=0.001905 -0.04706 -0.0120344 rpy=1.5708 1.5708 0 -> xyz=0.001905 -0.0638208 -0.0120344 rpy=1.5708 1.5708 0
- joint r3_p3_frame: origin xyz=-0.00508 -0.04706 -0.0192853 rpy=1.5708 1.5708 0 -> xyz=-0.00508 -0.0638208 -0.0192853 rpy=1.5708 1.5708 0
- joint r3_p4_frame: origin xyz=-0.00508 -0.04706 -0.0123397 rpy=1.5708 1.5708 0 -> xyz=-0.00508 -0.0638208 -0.0123397 rpy=1.5708 1.5708 0
